File: strobe.brd (EAGLE design)
At the start: 45.2 x 35.2 mm, 25 parts, among them Q1 2.5A/20V

Commit message: current version post print
Parts:
- renumbered U$1 to U1, U$10 to U8, U$11 to U11, U$12 to J1, U$13 to U2, U$2 to U6, U$3 to U7, U$4 to U9, U$5 to U10, U$6 to U12, U$7 to U4, U$8 to U3, U$9 to U5
Connections:
- net N$1 renamed GND
- net N$15 renamed LED_SW
- net N$17 renamed LED-
- net N$18 renamed VIN
- net N$2 renamed 5V
- net N$3 renamed SDA
- net N$4 renamed SCL
- net N$6 renamed U$
Other:
- board text added: "+"
- board text added: "-"
- board text added: "Apollo Robotic Systems"
- board text added: "Made By:"
- board text added: "SCL"
- board text added: "SDA"
- board text added: "Strobe Rev v0.1"
- board text added: "Taylor Dixon"
