File: strobe.sch (EAGLE design)
At the start: 25 parts, among them Q1 2.5A/20V

Commit message: current version post print
Parts:
- renumbered U$1 to U1, U$10 to U8, U$11 to U11, U$12 to J1, U$13 to U2, U$2 to U6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
Connections:
- net N$1 renamed GND
- net N$15 renamed LED_SW
- net N$17 renamed LED-
- net N$18 renamed VIN
- net N$2 renamed 5V
- net N$3 renamed SDA
- net N$4 renamed SCL
- net N$6 renamed U$
Other:
- note added: "J1"
- note added: "U1"
- note added: "U2"
